Commit message: renamed files

File: urdf/serpent.urdf (robot description, URDF)
Before this commit: robot modulessai, 33 links, 32 joints
Links:
- link Slide_key_joint_single1: geometry collision mesh filename=package://serpent_gazebo/meshes/Slide_key_joint_single1.STL; visual mesh filename=package://serpent_gazebo/meshes/Slide_key_joint_single1.STL
- link Slide_key_joint_single2: geometry collision mesh filename=package://serpent_gazebo/meshes/Slide_key_joint_single2.STL; visual mesh filename=package://serpent_gazebo/meshes/Slide_key_joint_single2.STL
- link joint_enclosure1: geometry collision mesh filename=package://serpent_gazebo/meshes/joint_enclosure1.STL; visual mesh filename=package://serpent_gazebo/meshes/joint_enclosure1.STL
- link joint_enclosure2: geometry collision mesh filename=package://serpent_gazebo/meshes/joint_enclosure2.STL; visual mesh filename=package://serpent_gazebo/meshes/joint_enclosure2.STL
- link scale1: geometry collision mesh filename=package://serpent_gazebo/meshes/scale1.STL; visual mesh filename=package://serpent_gazebo/meshes/scale1.STL
- link scale10: geometry collision mesh filename=package://serpent_gazebo/meshes/scale10.STL; visual mesh filename=package://serpent_gazebo/meshes/scale10.STL
- link scale11: geometry collision mesh filename=package://serpent_gazebo/meshes/scale11.STL; visual mesh filename=package://serpent_gazebo/meshes/scale11.STL
- link scale12: geometry collision mesh filename=package://serpent_gazebo/meshes/scale12.STL; visual mesh filename=package://serpent_gazebo/meshes/scale12.STL
- link scale13: geometry collision mesh filename=package://serpent_gazebo/meshes/scale13.STL; visual mesh filename=package://serpent_gazebo/meshes/scale13.STL
- link scale14: geometry collision mesh filename=package://serpent_gazebo/meshes/scale14.STL; visual mesh filename=package://serpent_gazebo/meshes/scale14.STL
- link scale15: geometry collision mesh filename=package://serpent_gazebo/meshes/scale15.STL; visual mesh filename=package://serpent_gazebo/meshes/scale15.STL
- link scale16: geometry collision mesh filename=package://serpent_gazebo/meshes/scale16.STL; visual mesh filename=package://serpent_gazebo/meshes/scale16.STL
- link scale2: geometry collision mesh filename=package://serpent_gazebo/meshes/scale2.STL; visual mesh filename=package://serpent_gazebo/meshes/scale2.STL
- link scale3: geometry collision mesh filename=package://serpent_gazebo/meshes/scale3.STL; visual mesh filename=package://serpent_gazebo/meshes/scale3.STL
- link scale4: geometry collision mesh filename=package://serpent_gazebo/meshes/scale4.STL; visual mesh filename=package://serpent_gazebo/meshes/scale4.STL
- link scale5: geometry collision mesh filename=package://serpent_gazebo/meshes/scale5.STL; visual mesh filename=package://serpent_gazebo/meshes/scale5.STL
- link scale6: geometry collision mesh filename=package://serpent_gazebo/meshes/scale6.STL; visual mesh filename=package://serpent_gazebo/meshes/scale6.STL
- link scale7: geometry collision mesh filename=package://serpent_gazebo/meshes/scale7.STL; visual mesh filename=package://serpent_gazebo/meshes/scale7.STL
- link scale8: geometry collision mesh filename=package://serpent_gazebo/meshes/scale8.STL; visual mesh filename=package://serpent_gazebo/meshes/scale8.STL
- link scale9: geometry collision mesh filename=package://serpent_gazebo/meshes/scale9.STL; visual mesh filename=package://serpent_gazebo/meshes/scale9.STL
- link shell1: geometry collision mesh filename=package://serpent_gazebo/meshes/shell1.STL; visual mesh filename=package://serpent_gazebo/meshes/shell1.STL
- link shell2: geometry collision mesh filename=package://serpent_gazebo/meshes/shell2.STL; visual mesh filename=package://serpent_gazebo/meshes/shell2.STL
- link slide_arm: geometry collision mesh filename=package://serpent_gazebo/meshes/slide_arm.STL; visual mesh filename=package://serpent_gazebo/meshes/slide_arm.STL
- link slide_arm2: geometry collision mesh filename=package://serpent_gazebo/meshes/slide_arm2.STL; visual mesh filename=package://serpent_gazebo/meshes/slide_arm2.STL
- link slide_clip1: geometry collision mesh filename=package://serpent_gazebo/meshes/slide_clip1.STL; visual mesh filename=package://serpent_gazebo/meshes/slide_clip1.STL
- link slide_clip2: geometry collision mesh filename=package://serpent_gazebo/meshes/slide_clip2.STL; visual mesh filename=package://serpent_gazebo/meshes/slide_clip2.STL
- link slide_clip3: geometry collision mesh filename=package://serpent_gazebo/meshes/slide_clip3.STL; visual mesh filename=package://serpent_gazebo/meshes/slide_clip3.STL
- link slide_clip4: geometry collision mesh filename=package://serpent_gazebo/meshes/slide_clip4.STL; visual mesh filename=package://serpent_gazebo/meshes/slide_clip4.STL
- link slide_key: geometry collision mesh filename=package://serpent_gazebo/meshes/slide_key.STL; visual mesh filename=package://serpent_gazebo/meshes/slide_key.STL
- link slide_key2: geometry collision mesh filename=package://serpent_gazebo/meshes/slide_key2.STL; visual mesh filename=package://serpent_gazebo/meshes/slide_key2.STL
- link slide_key_joint1: geometry collision mesh filename=package://serpent_gazebo/meshes/slide_key_joint1.STL; visual mesh filename=package://serpent_gazebo/meshes/slide_key_joint1.STL
- link slide_key_joint_2: geometry collision mesh filename=package://serpent_gazebo/meshes/slide_key_joint_2.STL; visual mesh filename=package://serpent_gazebo/meshes/slide_key_joint_2.STL
Joints:
- removed joint link9
- added joint serpent_main_joint: type continuous, parent shell1, child slide_key, origin xyz=-0.138611885720102 0.0896074988950939 -0.214616884182071 rpy=-1.5529323841969 0 -3.14159265358979, axis 0 0 0

Commit message: some work done but still not working

File: urdf/serpent.urdf (robot description, URDF)
Before this commit: robot serpent_gazebo, 33 links, 32 joints
Links:
- removed link base_footprint
- added link dummy
Joints:
- removed joint base_footprint_joint
- removed joint serpent_main_joint
- added joint dummy_joint: type fixed, parent dummy, child shell1
- added joint link9: type fixed, parent shell1, child slide_key, origin xyz=-0.138611885720102 0.0896074988950939 -0.214616884182071 rpy=-1.5529323841969 0 -3.14159265358979, axis 0 0 0
