Commit message: virtual model works as intended

File: urdf/serpent_old.urdf (robot description, URDF)
Before this commit: robot serpent, 4 links, 3 joints
Links:
- removed link base_link
- link TOP: mass 0.503745908624563 -> 0.503745908624564
Joints:
- removed joint base_link_to_chassis
- removed joint world_to_base_link
- added joint dummy_link: type fixed, parent world, child BOTTOM
- joint serpent_joint_1: origin xyz=0 -0.044432 0.15577 rpy=-1.8274 0 0 -> xyz=0 -0.044432012931505 -0.0505772211610462 rpy=1.31422119136425 0 -3.14159265358979
